Commit message: Escenas (payload/nopayload/motors/motors_nowall/gates) + wind_publisher + ExternalForce persistent
- Nuevo nodo wind_publisher (OU + Dryden + ráfagas)
- ExternalForce plugin: modo persistent + visualización
- Escenas: motors_gates, motors_nowall, nopayload, motors actualizadas
- Launch: args wind/turbulence/mean_wind_speed/wind_seed/gates_collide
- CLAUDE.md: documentación de escenas y perturbaciones

Co-Authored-By: Claude Opus 4.7 <noreply@anthropic.com>

File: src/acp_mujoco_simulator/model/quadrotor_acro_macro_motors.xml.xacro (robot description, xacro)
@@ -81,4 +81,16 @@
       <site name="${prefix}_payload_site" pos="0.0 0.0 -0.05"/>
       <camera name="${prefix}_camera" pos="0.035 0 -0.015" euler="0 0 -1.57"/>
+      <!-- Cinematic chase: hijo del body para que trackcom lo siga. Orientacion fija en mundo (sin roll/pitch). -->
+      <camera name="cinematic" mode="trackcom" pos="-3 -3 2" xyaxes="0.707 -0.707 0 0.304 0.304 0.906" fovy="70"/>
+      <!-- ═══════════════════════════════════════════════════════ -->
+      <!--  External wind/perturbation plugin (persistent mode).   -->
+      <!--  If no publisher on the topic, force stays zero.        -->
+      <!--  Activate with: ros2 run drone_teleop wind_publisher    -->
+      <!-- ═══════════════════════════════════════════════════════ -->
+      <plugin plugin="MujocoRosUtils::ExternalForce">
+        <config key="topic_name" value="/${prefix}/external_force"/>
+        <config key="vis_scale"  value="0.1"/>
+        <config key="persistent" value="true"/>
+      </plugin>
     </body>
   </xacro:macro>

File: src/acp_mujoco_simulator/model/scene_acro.xml.xacro (robot description, xacro)
@@ -47,4 +47,7 @@
     <geom name="origin_z" type="cylinder" fromto="0 0 0.01 0 0 0.51" size="0.01" rgba="0 0 1 0.1" contype="0" conaffinity="0" group="1"/>
     <camera name="camera_pov" pos="-2.427 1.392 1.622" xyaxes="-0.216 -0.976 -0.000 0.227 -0.050 0.973"/>
+    <!-- Cinematic tracking camera: follows drone position, does NOT rotate with it -->
+    <camera name="cinematic" mode="trackcom" target="$(arg quad_name)"
+            pos="0 -4 2" xyaxes="1 0 0 0 0.45 1"/>
   </worldbody>
   <actuator>

File: src/acp_mujoco_simulator/model/scene_acro_humanoid.xml.xacro (robot description, xacro)
@@ -50,4 +50,7 @@
     <geom name="origin_z" type="cylinder" fromto="0 0 0.01 0 0 0.51" size="0.01" rgba="0 0 1 0.1" contype="0" conaffinity="0" group="1"/>
     <camera name="camera_pov" pos="-2.427 1.392 1.622" xyaxes="-0.216 -0.976 -0.000 0.227 -0.050 0.973"/>
+    <!-- Cinematic tracking camera: follows drone position, does NOT rotate with it -->
+    <camera name="cinematic" mode="trackcom" target="$(arg quad_name)"
+            pos="0 -4 2" xyaxes="1 0 0 0 0.45 1"/>
   </worldbody>
   <actuator>

File: src/acp_mujoco_simulator/model/scene_acro_motors.xml.xacro (robot description, xacro)
@@ -20,4 +20,5 @@
     <plugin plugin="MujocoRosUtils::AcroMode"/>
     <plugin plugin="MujocoRosUtils::LowLevelMode"/>
+    <plugin plugin="MujocoRosUtils::ExternalForce"/>
   </extension>
   <asset>
@@ -51,4 +52,7 @@
     <geom name="origin_z" type="cylinder" fromto="0 0 0.01 0 0 0.51"   size="0.01" rgba="0 0 1 0.1" contype="0" conaffinity="0" group="1"/>
     <camera name="camera_pov" pos="-2.427 1.392 1.622" xyaxes="-0.216 -0.976 -0.000 0.227 -0.050 0.973"/>
+    <!-- Cinematic tracking camera: follows drone position, does NOT rotate with it -->
+    <camera name="cinematic" mode="trackcom" target="$(arg quad_name)"
+            pos="0 -4 2" xyaxes="1 0 0 0 0.45 1"/>
   </worldbody>
   <actuator>

File: src/acp_mujoco_simulator/model/scene_acro_motors_gates.xml.xacro (robot description, xacro)
@@ -9,4 +9,6 @@
   <xacro:arg name="init_pitch" default="0.0"/>
   <xacro:arg name="init_yaw"   default="0.0"/>
+  <xacro:arg name="gates_collide" default="0"/>
+  <xacro:property name="GATES_C" value="$(arg gates_collide)"/>
   <xacro:include filename="quadrotor_acro_macro_motors.xml.xacro" />
   <compiler angle="radian"/>
@@ -36,20 +38,20 @@
   <xacro:macro name="race_gate" params="name px py pz qw qx qy qz radius thickness material">
     <body name="${name}" pos="${px} ${py} ${pz}" quat="${qw} ${qx} ${qy} ${qz}">
-      <geom name="${name}_s00" type="capsule" fromto="0 +0.5000 +0.0000 0 +0.4619 +0.1913" size="${thickness}" material="${material}" contype="0" conaffinity="0"/>
-      <geom name="${name}_s01" type="capsule" fromto="0 +0.4619 +0.1913 0 +0.3536 +0.3536" size="${thickness}" material="${material}" contype="0" conaffinity="0"/>
-      <geom name="${name}_s02" type="capsule" fromto="0 +0.3536 +0.3536 0 +0.1913 +0.4619" size="${thickness}" material="${material}" contype="0" conaffinity="0"/>
-      <geom name="${name}_s03" type="capsule" fromto="0 +0.1913 +0.4619 0 +0.0000 +0.5000" size="${thickness}" material="${material}" contype="0" conaffinity="0"/>
-      <geom name="${name}_s04" type="capsule" fromto="0 +0.0000 +0.5000 0 -0.1913 +0.4619" size="${thickness}" material="${material}" contype="0" conaffinity="0"/>
-      <geom name="${name}_s05" type="capsule" fromto="0 -0.1913 +0.4619 0 -0.3536 +0.3536" size="${thickness}" material="${material}" contype="0" conaffinity="0"/>
-      <geom name="${name}_s06" type="capsule" fromto="0 -0.3536 +0.3536 0 -0.4619 +0.1913" size="${thickness}" material="${material}" contype="0" conaffinity="0"/>
-      <geom name="${name}_s07" type="capsule" fromto="0 -0.4619 +0.1913 0 -0.5000 +0.0000" size="${thickness}" material="${material}" contype="0" conaffinity="0"/>
-      <geom name="${name}_s08" type="capsule" fromto="0 -0.5000 +0.0000 0 -0.4619 -0.1913" size="${thickness}" material="${material}" contype="0" conaffinity="0"/>
-      <geom name="${name}_s09" type="capsule" fromto="0 -0.4619 -0.1913 0 -0.3536 -0.3536" size="${thickness}" material="${material}" contype="0" conaffinity="0"/>
-      <geom name="${name}_s10" type="capsule" fromto="0 -0.3536 -0.3536 0 -0.1913 -0.4619" size="${thickness}" material="${material}" contype="0" conaffinity="0"/>
-      <geom name="${name}_s11" type="capsule" fromto="0 -0.1913 -0.4619 0 -0.0000 -0.5000" size="${thickness}" material="${material}" contype="0" conaffinity="0"/>
-      <geom name="${name}_s12" type="capsule" fromto="0 -0.0000 -0.5000 0 +0.1913 -0.4619" size="${thickness}" material="${material}" contype="0" conaffinity="0"/>
-      <geom name="${name}_s13" type="capsule" fromto="0 +0.1913 -0.4619 0 +0.3536 -0.3536" size="${thickness}" material="${material}" contype="0" conaffinity="0"/>
-      <geom name="${name}_s14" type="capsule" fromto="0 +0.3536 -0.3536 0 +0.4619 -0.1913" size="${thickness}" material="${material}" contype="0" conaffinity="0"/>
-      <geom name="${name}_s15" type="capsule" fromto="0 +0.4619 -0.1913 0 +0.5000 -0.0000" size="${thickness}" material="${material}" contype="0" conaffinity="0"/>
+      <geom name="${name}_s00" type="capsule" fromto="0 +0.5000 +0.0000 0 +0.4619 +0.1913" size="${thickness}" material="${material}" contype="${GATES_C}" conaffinity="${GATES_C}"/>
+      <geom name="${name}_s01" type="capsule" fromto="0 +0.4619 +0.1913 0 +0.3536 +0.3536" size="${thickness}" material="${material}" contype="${GATES_C}" conaffinity="${GATES_C}"/>
+      <geom name="${name}_s02" type="capsule" fromto="0 +0.3536 +0.3536 0 +0.1913 +0.4619" size="${thickness}" material="${material}" contype="${GATES_C}" conaffinity="${GATES_C}"/>
+      <geom name="${name}_s03" type="capsule" fromto="0 +0.1913 +0.4619 0 +0.0000 +0.5000" size="${thickness}" material="${material}" contype="${GATES_C}" conaffinity="${GATES_C}"/>
+      <geom name="${name}_s04" type="capsule" fromto="0 +0.0000 +0.5000 0 -0.1913 +0.4619" size="${thickness}" material="${material}" contype="${GATES_C}" conaffinity="${GATES_C}"/>
+      <geom name="${name}_s05" type="capsule" fromto="0 -0.1913 +0.4619 0 -0.3536 +0.3536" size="${thickness}" material="${material}" contype="${GATES_C}" conaffinity="${GATES_C}"/>
+      <geom name="${name}_s06" type="capsule" fromto="0 -0.3536 +0.3536 0 -0.4619 +0.1913" size="${thickness}" material="${material}" contype="${GATES_C}" conaffinity="${GATES_C}"/>
+      <geom name="${name}_s07" type="capsule" fromto="0 -0.4619 +0.1913 0 -0.5000 +0.0000" size="${thickness}" material="${material}" contype="${GATES_C}" conaffinity="${GATES_C}"/>
+      <geom name="${name}_s08" type="capsule" fromto="0 -0.5000 +0.0000 0 -0.4619 -0.1913" size="${thickness}" material="${material}" contype="${GATES_C}" conaffinity="${GATES_C}"/>
+      <geom name="${name}_s09" type="capsule" fromto="0 -0.4619 -0.1913 0 -0.3536 -0.3536" size="${thickness}" material="${material}" contype="${GATES_C}" conaffinity="${GATES_C}"/>
+      <geom name="${name}_s10" type="capsule" fromto="0 -0.3536 -0.3536 0 -0.1913 -0.4619" size="${thickness}" material="${material}" contype="${GATES_C}" conaffinity="${GATES_C}"/>
+      <geom name="${name}_s11" type="capsule" fromto="0 -0.1913 -0.4619 0 -0.0000 -0.5000" size="${thickness}" material="${material}" contype="${GATES_C}" conaffinity="${GATES_C}"/>
+      <geom name="${name}_s12" type="capsule" fromto="0 -0.0000 -0.5000 0 +0.1913 -0.4619" size="${thickness}" material="${material}" contype="${GATES_C}" conaffinity="${GATES_C}"/>
+      <geom name="${name}_s13" type="capsule" fromto="0 +0.1913 -0.4619 0 +0.3536 -0.3536" size="${thickness}" material="${material}" contype="${GATES_C}" conaffinity="${GATES_C}"/>
+      <geom name="${name}_s14" type="capsule" fromto="0 +0.3536 -0.3536 0 +0.4619 -0.1913" size="${thickness}" material="${material}" contype="${GATES_C}" conaffinity="${GATES_C}"/>
+      <geom name="${name}_s15" type="capsule" fromto="0 +0.4619 -0.1913 0 +0.5000 -0.0000" size="${thickness}" material="${material}" contype="${GATES_C}" conaffinity="${GATES_C}"/>
     </body>
   </xacro:macro>
@@ -98,7 +100,8 @@
                      qw="+0.9743" qx="+0.0206" qy="-0.1001" qz="+0.2007"
                      radius="0.5" thickness="0.025" material="mat_gate_b"/>
-    <camera name="camera_pov" pos="-2.5 -3.0 2.5" xyaxes="0.95 -0.30 0 0.10 0.30 0.95"/>
-    <camera name="cinematic" mode="trackcom" target="$(arg quad_name)"
-            pos="0 -5 2.5" xyaxes="1 0 0 0 0.45 1"/>
+    <!-- camara `cinematic` chase definida dentro del macro del dron (hijo de body para track funcionar) -->
+    <!-- Spectator: parado en el suelo al costado (mitad de X, borde Y=-2), gira la cabeza para mirar al dron -->
+    <camera name="spectator" mode="targetbody" target="$(arg quad_name)"
+            pos="2.5 -1.95 1.7" fovy="75"/>
   </worldbody>
   <actuator>

File: src/acp_mujoco_simulator/model/scene_acro_motors_nowall.xml.xacro (robot description, xacro)
@@ -19,4 +19,5 @@
     <plugin plugin="MujocoRosUtils::AcroMode"/>
     <plugin plugin="MujocoRosUtils::LowLevelMode"/>
+    <plugin plugin="MujocoRosUtils::ExternalForce"/>
   </extension>
   <asset>
@@ -41,4 +42,7 @@
     <geom name="origin_z" type="cylinder" fromto="0 0 0.01 0 0 0.51"   size="0.01" rgba="0 0 1 0.1" contype="0" conaffinity="0" group="1"/>
     <camera name="camera_pov" pos="-2.427 1.392 1.622" xyaxes="-0.216 -0.976 -0.000 0.227 -0.050 0.973"/>
+    <!-- Cinematic tracking camera: follows drone position, does NOT rotate with it -->
+    <camera name="cinematic" mode="trackcom" target="$(arg quad_name)"
+            pos="0 -4 2" xyaxes="1 0 0 0 0.45 1"/>
   </worldbody>
   <actuator>

File: src/acp_mujoco_simulator/model/scene_acro_nopayload.xml.xacro (robot description, xacro)
@@ -45,4 +45,7 @@
     <geom name="origin_z" type="cylinder" fromto="0 0 0.01 0 0 0.51"   size="0.01" rgba="0 0 1 0.1" contype="0" conaffinity="0" group="1"/>
     <camera name="camera_pov" pos="-2.427 1.392 1.622" xyaxes="-0.216 -0.976 -0.000 0.227 -0.050 0.973"/>
+    <!-- Cinematic tracking camera: follows drone position, does NOT rotate with it -->
+    <camera name="cinematic" mode="trackcom" target="$(arg quad_name)"
+            pos="0 -4 2" xyaxes="1 0 0 0 0.45 1"/>
   </worldbody>
   <actuator>
